Commit message: modify .xacro file

File: nuturtle_description/urdf/turtlebot3_burger.urdf.xacro (robot description, xacro)
@@ -13,5 +13,5 @@
       <origin xyz="-0.032 0 0.0" rpy="0 0 0"/>
       <geometry>
-        <mesh filename="package://turtlebot3_description/meshes/bases/burger_base.stl" scale="0.001 0.001 0.001"/>
+        <mesh filename="package://nuturtlebot_description/meshes/burger_base.stl" scale="0.001 0.001 0.001"/>
       </geometry>
       <material name="light_black"/>
@@ -41,5 +41,5 @@
       <origin xyz="0 0 0" rpy="1.57 0 0"/>
       <geometry>
-        <mesh filename="package://turtlebot3_description/meshes/wheels/left_tire.stl" scale="0.001 0.001 0.001"/>
+        <mesh filename="package://nuturtlebot_description/meshes/left_tire.stl" scale="0.001 0.001 0.001"/>
       </geometry>
       <material name="dark"/>
@@ -69,5 +69,5 @@
       <origin xyz="0 0 0" rpy="1.57 0 0"/>
       <geometry>
-        <mesh filename="package://turtlebot3_description/meshes/wheels/right_tire.stl" scale="0.001 0.001 0.001"/>
+        <mesh filename="package://nuturtlebot_description/meshes/right_tire.stl" scale="0.001 0.001 0.001"/>
       </geometry>
       <material name="dark"/>
@@ -122,5 +122,5 @@
       <origin xyz="0 0 0.0" rpy="0 0 0"/>
       <geometry>
-        <mesh filename="package://turtlebot3_description/meshes/sensors/lds.stl" scale="0.001 0.001 0.001"/>
+        <mesh filename="package://nuturtlebot_description/meshes/lds.stl" scale="0.001 0.001 0.001"/>
       </geometry>
       <material name="dark"/>

Commit message: create diff_params.yaml

File: nuturtle_description/urdf/turtlebot3_burger.urdf.xacro (robot description, xacro)
@@ -1,6 +1,6 @@
 <?xml version="1.0" ?>
 <robot name="turtlebot3_burger" xmlns:xacro="http://ros.org/wiki/xacro">
-  <xacro:include filename="$(find nuturtlebot_description)/urdf/common_properties.xacro"/>
-  <xacro:include filename="$(find nuturtlebot_description)/urdf/turtlebot3_burger.gazebo.xacro"/>
+  <xacro:include filename="$(find nuturtle_description)/urdf/common_properties.xacro"/>
+  <xacro:include filename="$(find nuturtle_description)/urdf/turtlebot3_burger.gazebo.xacro"/>
   <link name="base_footprint"/>
   <joint name="base_joint" type="fixed">
@@ -13,5 +13,5 @@
       <origin xyz="-0.032 0 0.0" rpy="0 0 0"/>
       <geometry>
-        <mesh filename="package://nuturtlebot_description/meshes/burger_base.stl" scale="0.001 0.001 0.001"/>
+        <mesh filename="package://nuturtle_description/meshes/burger_base.stl" scale="0.001 0.001 0.001"/>
       </geometry>
       <material name="light_black"/>
@@ -41,5 +41,5 @@
       <origin xyz="0 0 0" rpy="1.57 0 0"/>
       <geometry>
-        <mesh filename="package://nuturtlebot_description/meshes/left_tire.stl" scale="0.001 0.001 0.001"/>
+        <mesh filename="package://nuturtle_description/meshes/left_tire.stl" scale="0.001 0.001 0.001"/>
       </geometry>
       <material name="dark"/>
@@ -69,5 +69,5 @@
       <origin xyz="0 0 0" rpy="1.57 0 0"/>
       <geometry>
-        <mesh filename="package://nuturtlebot_description/meshes/right_tire.stl" scale="0.001 0.001 0.001"/>
+        <mesh filename="package://nuturtle_description/meshes/right_tire.stl" scale="0.001 0.001 0.001"/>
       </geometry>
       <material name="dark"/>
@@ -122,5 +122,5 @@
       <origin xyz="0 0 0.0" rpy="0 0 0"/>
       <geometry>
-        <mesh filename="package://nuturtlebot_description/meshes/lds.stl" scale="0.001 0.001 0.001"/>
+        <mesh filename="package://nuturtle_description/meshes/lds.stl" scale="0.001 0.001 0.001"/>
       </geometry>
       <material name="dark"/>

Commit message: add arg color

File: nuturtle_description/urdf/turtlebot3_burger.urdf.xacro (robot description, xacro)
@@ -3,4 +3,12 @@
   <xacro:include filename="$(find nuturtle_description)/urdf/common_properties.xacro"/>
   <xacro:include filename="$(find nuturtle_description)/urdf/turtlebot3_burger.gazebo.xacro"/>
+  <!-- load yaml file and two parameters-->
+  <xacro:property name='yaml_file' value='$(find nuturtle_description)/config/diff_params.yaml'/>
+  <xacro:property name='diff_params' value='${load_yaml(yaml_file)}'/>
+  <xacro:property name= "wheel_radius" value="${diff_params['wheel_radius']}"/>
+  <xacro:property name= "track_width" value="${diff_params['track_width']}"/>
+  <!-- <xacro:property name="color" value="black"/> -->
+  <xacro:arg name="color" default = "black"/>
+  <!-- <xacro:property name="colour" value="$(arg color)"/> -->
   <link name="base_footprint"/>
   <joint name="base_joint" type="fixed">
@@ -15,5 +23,5 @@
         <mesh filename="package://nuturtle_description/meshes/burger_base.stl" scale="0.001 0.001 0.001"/>
       </geometry>
-      <material name="light_black"/>
+      <material name="$(arg color)"/>
     </visual>
     <collision>
@@ -34,5 +42,5 @@
     <parent link="base_link"/>
     <child link="wheel_left_link"/>
-    <origin xyz="0.0 0.08 0.023" rpy="-1.57 0 0"/>
+    <origin xyz="0.0 ${track_width/2} 0.023" rpy="-1.57 0 0"/>
     <axis xyz="0 0 1"/>
   </joint>
@@ -48,5 +56,5 @@
       <origin xyz="0 0 0" rpy="0 0 0"/>
       <geometry>
-        <cylinder length="0.018" radius="0.033"/>
+        <cylinder length="0.018" radius="${wheel_radius}"/>
       </geometry>
     </collision>
@@ -62,5 +70,5 @@
     <parent link="base_link"/>
     <child link="wheel_right_link"/>
-    <origin xyz="0.0 -0.080 0.023" rpy="-1.57 0 0"/>
+    <origin xyz="0.0 ${-track_width/2} 0.023" rpy="-1.57 0 0"/>
     <axis xyz="0 0 1"/>
   </joint>
@@ -76,5 +84,5 @@
       <origin xyz="0 0 0" rpy="0 0 0"/>
       <geometry>
-        <cylinder length="0.018" radius="0.033"/>
+        <cylinder length="0.018" radius="${wheel_radius}"/>
       </geometry>
     </collision>

Commit message: finish task a4

File: nuturtle_description/urdf/turtlebot3_burger.urdf.xacro (robot description, xacro)
@@ -8,14 +8,13 @@
   <xacro:property name= "wheel_radius" value="${diff_params['wheel_radius']}"/>
   <xacro:property name= "track_width" value="${diff_params['track_width']}"/>
-  <!-- <xacro:property name="color" value="black"/> -->
+  <!-- pass arg from launch file to here-->
   <xacro:arg name="color" default = "black"/>
-  <!-- <xacro:property name="colour" value="$(arg color)"/> -->
-  <link name="base_footprint"/>
-  <joint name="base_joint" type="fixed">
-    <parent link="base_footprint"/>
-    <child link="base_link"/>
+  <link name="$(arg color)/base_footprint"/>
+  <joint name="$(arg color)/base_joint" type="fixed">
+    <parent link="$(arg color)/base_footprint"/>
+    <child link="$(arg color)/base_link"/>
     <origin xyz="0.0 0.0 0.010" rpy="0 0 0"/>
   </joint>
-  <link name="base_link">
+  <link name="$(arg color)/base_link">
     <visual>
       <origin xyz="-0.032 0 0.0" rpy="0 0 0"/>
@@ -39,11 +38,11 @@
     </inertial>
   </link>
-  <joint name="wheel_left_joint" type="continuous">
-    <parent link="base_link"/>
-    <child link="wheel_left_link"/>
+  <joint name="$(arg color)/wheel_left_joint" type="continuous">
+    <parent link="$(arg color)/base_link"/>
+    <child link="$(arg color)/wheel_left_link"/>
     <origin xyz="0.0 ${track_width/2} 0.023" rpy="-1.57 0 0"/>
     <axis xyz="0 0 1"/>
   </joint>
-  <link name="wheel_left_link">
+  <link name="$(arg color)/wheel_left_link">
     <visual>
       <origin xyz="0 0 0" rpy="1.57 0 0"/>
@@ -67,11 +66,11 @@
       </inertial>
   </link>
-  <joint name="wheel_right_joint" type="continuous">
-    <parent link="base_link"/>
-    <child link="wheel_right_link"/>
+  <joint name="$(arg color)/wheel_right_joint" type="continuous">
+    <parent link="$(arg color)/base_link"/>
+    <child link="$(arg color)/wheel_right_link"/>
     <origin xyz="0.0 ${-track_width/2} 0.023" rpy="-1.57 0 0"/>
     <axis xyz="0 0 1"/>
   </joint>
-  <link name="wheel_right_link">
+  <link name="$(arg color)/wheel_right_link">
     <visual>
       <origin xyz="0 0 0" rpy="1.57 0 0"/>
@@ -95,10 +94,10 @@
       </inertial>
   </link>
-  <joint name="caster_back_joint" type="fixed">
-    <parent link="base_link"/>
-    <child link="caster_back_link"/>
+  <joint name="$(arg color)/caster_back_joint" type="fixed">
+    <parent link="$(arg color)/base_link"/>
+    <child link="$(arg color)/caster_back_link"/>
     <origin xyz="-0.081 0 -0.004" rpy="-1.57 0 0"/>
   </joint>
-  <link name="caster_back_link">
+  <link name="$(arg color)/caster_back_link">
     <collision>
       <origin xyz="0 0.001 0" rpy="0 0 0"/>
@@ -115,16 +114,16 @@
     </inertial>
   </link>
-  <joint name="imu_joint" type="fixed">
-    <parent link="base_link"/>
-    <child link="imu_link"/>
+  <joint name="$(arg color)/imu_joint" type="fixed">
+    <parent link="$(arg color)/base_link"/>
+    <child link="$(arg color)/imu_link"/>
     <origin xyz="-0.032 0 0.068" rpy="0 0 0"/>
   </joint>
-  <link name="imu_link"/>
-  <joint name="scan_joint" type="fixed">
-    <parent link="base_link"/>
-    <child link="base_scan"/>
+  <link name="$(arg color)/imu_link"/>
+  <joint name="$(arg color)/scan_joint" type="fixed">
+    <parent link="$(arg color)/base_link"/>
+    <child link="$(arg color)/base_scan"/>
     <origin xyz="-0.032 0 0.172" rpy="0 0 0"/>
   </joint>
-  <link name="base_scan">
+  <link name="$(arg color)/base_scan">
     <visual>
       <origin xyz="0 0 0.0" rpy="0 0 0"/>

Commit message: create frame_main.cpp

File: nuturtle_description/urdf/turtlebot3_burger.urdf.xacro (robot description, xacro)
@@ -10,11 +10,11 @@
   <!-- pass arg from launch file to here-->
   <xacro:arg name="color" default = "black"/>
-  <link name="$(arg color)/base_footprint"/>
-  <joint name="$(arg color)/base_joint" type="fixed">
-    <parent link="$(arg color)/base_footprint"/>
-    <child link="$(arg color)/base_link"/>
+  <link name="$(arg color)-base_footprint"/>
+  <joint name="$(arg color)-base_joint" type="fixed">
+    <parent link="$(arg color)-base_footprint"/>
+    <child link="$(arg color)-base_link"/>
     <origin xyz="0.0 0.0 0.010" rpy="0 0 0"/>
   </joint>
-  <link name="$(arg color)/base_link">
+  <link name="$(arg color)-base_link">
     <visual>
       <origin xyz="-0.032 0 0.0" rpy="0 0 0"/>
@@ -38,11 +38,11 @@
     </inertial>
   </link>
-  <joint name="$(arg color)/wheel_left_joint" type="continuous">
-    <parent link="$(arg color)/base_link"/>
-    <child link="$(arg color)/wheel_left_link"/>
+  <joint name="$(arg color)-wheel_left_joint" type="continuous">
+    <parent link="$(arg color)-base_link"/>
+    <child link="$(arg color)-wheel_left_link"/>
     <origin xyz="0.0 ${track_width/2} 0.023" rpy="-1.57 0 0"/>
     <axis xyz="0 0 1"/>
   </joint>
-  <link name="$(arg color)/wheel_left_link">
+  <link name="$(arg color)-wheel_left_link">
     <visual>
       <origin xyz="0 0 0" rpy="1.57 0 0"/>
@@ -66,11 +66,11 @@
       </inertial>
   </link>
-  <joint name="$(arg color)/wheel_right_joint" type="continuous">
-    <parent link="$(arg color)/base_link"/>
-    <child link="$(arg color)/wheel_right_link"/>
+  <joint name="$(arg color)-wheel_right_joint" type="continuous">
+    <parent link="$(arg color)-base_link"/>
+    <child link="$(arg color)-wheel_right_link"/>
     <origin xyz="0.0 ${-track_width/2} 0.023" rpy="-1.57 0 0"/>
     <axis xyz="0 0 1"/>
   </joint>
-  <link name="$(arg color)/wheel_right_link">
+  <link name="$(arg color)-wheel_right_link">
     <visual>
       <origin xyz="0 0 0" rpy="1.57 0 0"/>
@@ -94,10 +94,10 @@
       </inertial>
   </link>
-  <joint name="$(arg color)/caster_back_joint" type="fixed">
-    <parent link="$(arg color)/base_link"/>
-    <child link="$(arg color)/caster_back_link"/>
+  <joint name="$(arg color)-caster_back_joint" type="fixed">
+    <parent link="$(arg color)-base_link"/>
+    <child link="$(arg color)-caster_back_link"/>
     <origin xyz="-0.081 0 -0.004" rpy="-1.57 0 0"/>
   </joint>
-  <link name="$(arg color)/caster_back_link">
+  <link name="$(arg color)-caster_back_link">
     <collision>
       <origin xyz="0 0.001 0" rpy="0 0 0"/>
@@ -114,16 +114,16 @@
     </inertial>
   </link>
-  <joint name="$(arg color)/imu_joint" type="fixed">
-    <parent link="$(arg color)/base_link"/>
-    <child link="$(arg color)/imu_link"/>
+  <joint name="$(arg color)-imu_joint" type="fixed">
+    <parent link="$(arg color)-base_link"/>
+    <child link="$(arg color)-imu_link"/>
     <origin xyz="-0.032 0 0.068" rpy="0 0 0"/>
   </joint>
-  <link name="$(arg color)/imu_link"/>
-  <joint name="$(arg color)/scan_joint" type="fixed">
-    <parent link="$(arg color)/base_link"/>
-    <child link="$(arg color)/base_scan"/>
+  <link name="$(arg color)-imu_link"/>
+  <joint name="$(arg color)-scan_joint" type="fixed">
+    <parent link="$(arg color)-base_link"/>
+    <child link="$(arg color)-base_scan"/>
     <origin xyz="-0.032 0 0.172" rpy="0 0 0"/>
   </joint>
-  <link name="$(arg color)/base_scan">
+  <link name="$(arg color)-base_scan">
     <visual>
       <origin xyz="0 0 0.0" rpy="0 0 0"/>

Commit message: add collision radius

File: nuturtle_description/urdf/turtlebot3_burger.urdf.xacro (robot description, xacro)
@@ -3,9 +3,10 @@
   <xacro:include filename="$(find nuturtle_description)/urdf/common_properties.xacro"/>
   <xacro:include filename="$(find nuturtle_description)/urdf/turtlebot3_burger.gazebo.xacro"/>
-  <!-- load yaml file and two parameters-->
+  <!-- load yaml file and three parameters-->
   <xacro:property name='yaml_file' value='$(find nuturtle_description)/config/diff_params.yaml'/>
   <xacro:property name='diff_params' value='${load_yaml(yaml_file)}'/>
   <xacro:property name= "wheel_radius" value="${diff_params['wheel_radius']}"/>
   <xacro:property name= "track_width" value="${diff_params['track_width']}"/>
+  <xacro:property name= "collision_radius" value="${diff_params['collision_radius']}"/>
   <!-- pass arg from launch file to here-->
   <xacro:arg name="color" default = "black"/>

Commit message: urdf tweaks

File: nuturtle_description/urdf/turtlebot3_burger.urdf.xacro (robot description, xacro)
@@ -25,10 +25,20 @@
       <material name="$(arg color)"/>
     </visual>
-    <collision>
-      <origin xyz="-0.032 0 0.070" rpy="0 0 0"/>
-      <geometry>
-        <box size="0.140 0.140 0.143"/>
-      </geometry>
-    </collision>
+    <xacro:if value="${collision_radius == 0}">
+      <collision>
+        <origin xyz="-0.032 0 0.070" rpy="0 0 0"/>
+        <geometry>
+          <box size="0.140 0.140 0.143"/>
+        </geometry>
+      </collision>
+    </xacro:if>
+    <xacro:if value="${collision_radius != 0}">
+      <collision>
+        <origin xyz="-0.032 0 0.070" rpy="0 0 0"/>
+        <geometry>
+          <cylinder length="0.143" radius="${collision_radius}"/>
+        </geometry>
+      </collision>
+    </xacro:if>
     <inertial>
       <origin xyz="0 0 0" rpy="0 0 0"/>
